Commit message: dataset added for hook-tape; inference adapted; all dirs checked for compatibility

File: torch_robotics/data/urdf/objects/slatwall-hook/slatwall_hook.urdf (robot description, URDF)
Before this commit: robot hook, 1 links, 0 joints
Links:
- link base_link: mass 0.5 -> 1.0; geometry collision mesh filename=package://slatwall-hook/slatwall_vhacd.obj scale=0.002 0.002 0.002; visual mesh filename=package://slatwall-hook/slatwall.stl scale=0.002 0.002 0.002

File: torch_robotics/data/urdf/robots/rigid_3d/tape/tape.urdf (robot description, URDF)
Before this commit: robot donut, 1 links, 0 joints
Links:
- link base_link: mass 0.5 -> 1.0
